Commit message: changed gpu lidar specs to reflect that of livox mid360

File: go2_description/xacro/gazebo(mid).xacro (robot description, xacro)
@@ -99,43 +99,42 @@
                 </plugin>
                 <pose>0 0 0 0 0 0</pose>
-                <gz_frame_id>imu_link</gz_frame_id> <!-- Добавьте этот тег для указания кадра -->
+                <gz_frame_id>imu_link</gz_frame_id>
             </sensor>
         </gazebo>
         <gazebo reference="laser_frame">
-            <!--<material>Gazebo/Black</material>-->
-	<sensor name="laser" type="gpu_lidar">
-  <pose>0 0 0 0 0 0</pose>
-  <visualize>false</visualize>
-  <update_rate>10</update_rate>
-  <lidar>
-    <scan>
-      <horizontal>
-        <samples>1000</samples>
-        <resolution>1</resolution>
-        <min_angle>-3.14159</min_angle>
-        <max_angle>3.14159</max_angle>
-      </horizontal>
-      <vertical>
-        <samples>40</samples>
-        <resolution>1</resolution>
-        <min_angle>-0.12217</min_angle>
-        <max_angle>0.90757</max_angle>
-      </vertical>
-    </scan>
-    <range>
-      <min>0.1</min>
-      <max>40.0</max>
-      <resolution>0.01</resolution>
-    </range>
-    <noise>
-      <type>gaussian</type>
-      <mean>0.0</mean>
-      <stddev>0.01</stddev>
-    </noise>
-  </lidar>
-  <topic>/${robot_name}/points</topic>
-  <gz_frame_id>laser_frame</gz_frame_id>
-</sensor>
-</gazebo>
+            <sensor name="laser" type="gpu_lidar">
+                <pose>0 0 0 0 0 0</pose>
+                <visualize>false</visualize>
+                <update_rate>10</update_rate>
+                <lidar>
+                    <scan>
+                        <horizontal>
+                            <samples>1000</samples>
+                            <resolution>1</resolution>
+                            <min_angle>-3.14159265</min_angle>
+                            <max_angle>3.14159265</max_angle>
+                        </horizontal>
+                        <vertical>
+                            <samples>40</samples>
+                            <resolution>1</resolution>
+                            <min_angle>-0.12217305</min_angle>
+                            <max_angle>0.90757121</max_angle>
+                        </vertical>
+                    </scan>
+                    <range>
+                        <min>0.1</min>
+                        <max>40.0</max>
+                        <resolution>0.002</resolution>
+                    </range>
+                    <noise>
+                        <type>gaussian</type>
+                        <mean>0.0</mean>
+                        <stddev>0.01</stddev>
+                    </noise>
+                </lidar>
+                <topic>/${robot_name}/points/points</topic>
+                <gz_frame_id>laser_frame</gz_frame_id>
+            </sensor>
+        </gazebo>
         <gazebo reference="camera_face">
             <!-- <material>Gazebo/Black</material> -->
@@ -167,12 +166,4 @@
             <kd>1.0</kd>
         </gazebo>
-        <!-- <gazebo reference="stick_link">
-            <mu1>0.2</mu1>
-            <mu2>0.2</mu2>
-        </gazebo> -->
-        <!-- <gazebo reference="imu_link">
-            <mu1>0.2</mu1>
-            <mu2>0.2</mu2>
-        </gazebo> -->
         <!-- FL leg -->
         <gazebo reference="lf_hip_link">

Commit message: lidar mount and mid360

File: go2_description/xacro/gazebo(mid).xacro (robot description, xacro)
@@ -102,39 +102,40 @@
             </sensor>
         </gazebo>
-        <gazebo reference="laser_frame">
-            <sensor name="laser" type="gpu_lidar">
-                <pose>0 0 0 0 0 0</pose>
-                <visualize>false</visualize>
-                <update_rate>10</update_rate>
-                <lidar>
-                    <scan>
-                        <horizontal>
-                            <samples>1000</samples>
-                            <resolution>1</resolution>
-                            <min_angle>-3.14159265</min_angle>
-                            <max_angle>3.14159265</max_angle>
-                        </horizontal>
-                        <vertical>
-                            <samples>40</samples>
-                            <resolution>1</resolution>
-                            <min_angle>-0.12217305</min_angle>
-                            <max_angle>0.90757121</max_angle>
-                        </vertical>
-                    </scan>
-                    <range>
-                        <min>0.1</min>
-                        <max>40.0</max>
-                        <resolution>0.002</resolution>
-                    </range>
-                    <noise>
-                        <type>gaussian</type>
-                        <mean>0.0</mean>
-                        <stddev>0.01</stddev>
-                    </noise>
-                </lidar>
-                <topic>/${robot_name}/points/points</topic>
-                <gz_frame_id>laser_frame</gz_frame_id>
-            </sensor>
-        </gazebo>
+	<gazebo reference="laser_frame">
+	    <sensor name="gpu_lidar" type="gpu_lidar">
+		<pose relative_to="laser_frame">0 0 0 0 0 0</pose>
+		<topic>/${robot_name}/points/points</topic>
+		<update_rate>10</update_rate>
+		<lidar>
+		    <scan>
+		        <horizontal>
+		            <samples>720</samples>
+		            <resolution>1</resolution>
+		            <min_angle>-3.14159265</min_angle>
+		            <max_angle>3.14159265</max_angle>
+		        </horizontal>
+		        <vertical>
+		            <samples>40</samples>
+		            <resolution>1</resolution>
+		            <min_angle>0</min_angle>
+		            <max_angle>0.9774</max_angle>
+		        </vertical>
+		    </scan>
+		    <range>
+		        <min>0.01</min>
+		        <max>40.0</max>
+		        <resolution>0.01</resolution>
+		    </range>
+		    <noise>
+		        <type>gaussian</type>
+		        <mean>0.0</mean>
+		        <stddev>0.01</stddev>
+		    </noise>
+		</lidar>
+		<always_on>1</always_on>
+		<visualize>false</visualize>
+		<gz_frame_id>laser_frame</gz_frame_id>
+	    </sensor>
+	</gazebo>
         <gazebo reference="camera_face">
             <!-- <material>Gazebo/Black</material> -->

File: go2_description/xacro/robot.xacro (robot description, xacro)
@@ -60,26 +60,19 @@
         <parent link="base_link"/>
         <child link="laser_frame"/>
-        <origin xyz="0.22 0.0 0.095" rpy="0 0 0" />
+        <origin xyz="0.035 0.02 0.065" rpy="0 0 0" />
     </joint>
-    <link name="laser_frame">
-        <inertial>
-            <mass value="0.001"/>
-            <origin rpy="0 0 0" xyz="0 0 0"/>
-            <inertia ixx="0.0001" ixy="0" ixz="0" iyy="0.0001" iyz="0" izz="0.0001"/>
-        </inertial>
-        <visual>
-            <origin rpy="0 0 0" xyz="0 0 0"/>
-            <geometry>
-                <cylinder length="0.01" radius="0.018" />
-            </geometry>
-            <!-- <material name="red"/> -->
-        </visual>
-        <collision>
-            <origin rpy="0 0 0" xyz="0 0 0"/>
-            <geometry>
-                <cylinder length="0.01" radius="0.018" />
-            </geometry>
-        </collision>
-    </link>
+	<link name="laser_frame">
+	    <visual>
+		<origin xyz="0 0 0" rpy="${3*pi/2} ${pi} ${3*pi/2}"/>
+		<geometry>
+		    <mesh filename="file://$(find go2_description)/meshes/avengers_endgame.glb" scale="0.055 0.055 0.055"/>
+		</geometry>
+	    </visual>
+	    <inertial>
+		<mass value="0.265"/>
+		<origin xyz="0 0 0" rpy="0 0 0"/>
+		<inertia ixx="0.0001" ixy="0" ixz="0" iyy="0.0001" iyz="0" izz="0.0001"/>
+	    </inertial>
+	</link>
     <joint name="imu_joint" type="fixed">
         <parent link="base_link"/>
