Commit message: 3d lidar data

File: go2_description/xacro/gazebo.xacro (robot description, xacro)
@@ -104,24 +104,29 @@
         <gazebo reference="laser_frame">
             <!--<material>Gazebo/Black</material>-->
-            <sensor name="laser" type="gpu_lidar">
-                <pose> 0 0 0 0 0 0 </pose>
-                <visualize>false</visualize>
-                <update_rate>10</update_rate>
-                <lidar>
-                    <scan>
-                        <horizontal>
-                            <samples>360</samples>
-                            <min_angle>-3.14</min_angle>
-                            <max_angle>3.14</max_angle>
-                        </horizontal>
-                    </scan>
-                    <range>
-                        <min>0.05</min>
-                        <max>12</max>
-                    </range>
-                </lidar>
-                <topic>/${robot_name}/scan</topic>
-                <gz_frame_id>laser_frame</gz_frame_id>
-            </sensor>
+	<sensor name="laser" type="gpu_lidar">
+	    <pose> 0 0 0 0 0 0 </pose>
+	    <visualize>false</visualize>
+	    <update_rate>10</update_rate>
+	    <lidar>
+	        <scan>
+	            <horizontal>
+	                <samples>360</samples>
+	                <min_angle>-3.14</min_angle>
+	                <max_angle>3.14</max_angle>
+	            </horizontal>
+	            <vertical>
+	                <samples>16</samples>
+	                <min_angle>-0.2618</min_angle>
+	                <max_angle>0.2618</max_angle>
+	            </vertical>
+	        </scan>
+	        <range>
+	            <min>0.05</min>
+	            <max>12</max>
+	        </range>
+	    </lidar>
+	    <topic>/${robot_name}/points</topic>
+	    <gz_frame_id>laser_frame</gz_frame_id>
+	</sensor>
         </gazebo>
         <gazebo reference="camera_face">

File: go2_description/xacro/robot.xacro (robot description, xacro)
@@ -58,5 +58,5 @@
     </link>
     <joint name='laser_scan' type='fixed'>
-        <parent link="base_link"/>,
+        <parent link="base_link"/>
         <child link="laser_frame"/>
         <origin xyz="0.22 0.0 0.095" rpy="0 0 0" />

Commit message: glim map generated, mid360 lidar

File: go2_description/xacro/gazebo.xacro (robot description, xacro)
@@ -102,39 +102,18 @@
             </sensor>
         </gazebo>
-        <gazebo reference="laser_frame">
-            <!--<material>Gazebo/Black</material>-->
-	<sensor name="laser" type="gpu_lidar">
-  <pose>0 0 0 0 0 0</pose>
-  <visualize>false</visualize>
-  <update_rate>10</update_rate>
-  <lidar>
-    <scan>
-      <horizontal>
-        <samples>1000</samples>
-        <resolution>1</resolution>
-        <min_angle>-3.14159</min_angle>
-        <max_angle>3.14159</max_angle>
-      </horizontal>
-      <vertical>
-        <samples>40</samples>
-        <resolution>1</resolution>
-        <min_angle>-0.12217</min_angle>
-        <max_angle>0.90757</max_angle>
-      </vertical>
-    </scan>
-    <range>
-      <min>0.1</min>
-      <max>40.0</max>
-      <resolution>0.01</resolution>
-    </range>
-    <noise>
-      <type>gaussian</type>
-      <mean>0.0</mean>
-      <stddev>0.01</stddev>
-    </noise>
-  </lidar>
-  <topic>/${robot_name}/points</topic>
-  <gz_frame_id>laser_frame</gz_frame_id>
-</sensor>
+	<gazebo reference="laser_frame">
+    <sensor name="mid360" type="custom">
+        <plugin filename="RGLServerPluginInstance" name="rgl::RGLServerPluginInstance">
+            <range>
+                <min>0.1</min>
+                <max>40.0</max>
+            </range>
+            <update_rate>10</update_rate>
+            <update_on_paused_sim>false</update_on_paused_sim>
+            <topic>/robot1/points/points_timed</topic>
+            <frame>laser_frame</frame>
+            <pattern_preset_path>/rgl_patterns/LivoxMid360.mat3x4f</pattern_preset_path>
+        </plugin>
+    </sensor>
 </gazebo>
         <gazebo reference="camera_face">
